Commit message: debug training part, add collision check. 1. debug DDPG.py, arm_env.py, simulate_state.py, etc; 2. add moveit collision detection.

File: as_arm_description/urdf/as_arm.urdf (robot description, URDF)
Before this commit: robot as_arm, 19 links, 18 joints
Links:
- added link world
Joints:
- added joint world_joint: type fixed, parent world, child base_link, origin xyz=0 0 0.04 rpy=0 0 0

File: as_arm_description/urdf/as_arm.xacro (robot description, xacro)
@@ -32,12 +32,18 @@
             <type>transmission_interface/SimpleTransmission</type>
             <joint name="${joint_name}">
-                <hardwareInterface>PositionJointInterface</hardwareInterface>
+                <hardwareInterface>EffortJointInterface</hardwareInterface>
             </joint>
             <actuator name="motor1">
-                <hardwareInterface>PositionJointInterface</hardwareInterface>
+                <hardwareInterface>EffortJointInterface</hardwareInterface>
                 <mechanicalReduction>1</mechanicalReduction>
             </actuator>
         </transmission>
     </xacro:macro>
+    <link name="world"/>
+    <joint name="world_joint" type="fixed">
+        <origin xyz="0 0 0.04" rpy="0 0 0"/>
+        <parent link="world"/>
+        <child link="base_link"/>
+    </joint>
     <!-- ////  bottom link -> base link  ////-->
     <link name="bottom_link">
@@ -257,5 +263,5 @@
         <origin xyz="0 0 0.002"/>
         <axis xyz="0 1 0"/>
-        <limit effort="100" lower="-0.015" upper="0" velocity="1.0"/>
+        <limit effort="200" lower="-0.015" upper="0" velocity="1.0"/>
         <dynamics damping="50" friction="1"/>
     </joint>
@@ -268,5 +274,5 @@
             <material name="Black"/>
         </visual>
-        <xacro:inertial_matrix mass="1"/>
+        <xacro:inertial_matrix mass="0.2"/>
     </link>
     <gazebo reference="l_gripper_aft_link">
@@ -279,5 +285,5 @@
         <origin xyz="0 0 0.002"/>
         <axis xyz="0 1 0"/>
-        <limit effort="100" lower="0" upper="0.015" velocity="1.0"/>
+        <limit effort="200" lower="0" upper="0.015" velocity="1.0"/>
         <dynamics damping="50" friction="1"/>
     </joint>
@@ -290,5 +296,5 @@
             <material name="Black"/>
         </visual>
-        <xacro:inertial_matrix mass="1"/>
+        <xacro:inertial_matrix mass="0.2"/>
     </link>
     <gazebo reference="r_gripper_aft_link">
@@ -315,4 +321,5 @@
         <child link="grasp_frame_link"/>
         <origin xyz="0 0 0.065" rpy="0 0 0"/>
+        <!--limit effort="300" velocity="1" lower="0" upper="0"/-->
     </joint>
     <!-- transmission block -->

File: as_arm_description/urdf/camera.xacro (robot description, xacro)
@@ -16,5 +16,5 @@
         </visual>
         <collision>
-            <origin xyz=" 0 0 ${MAST_HEIGHT-0.02}" rpy="0 0 0"/>
+            <origin xyz=" 0 0 ${MAST_HEIGHT/2-0.02}" rpy="0 0 0"/>
             <geometry>
                 <box size="0.01 0.01 ${MAST_HEIGHT}"/>

File: as_arm_description/urdf/object.xacro (robot description, xacro)
@@ -9,5 +9,5 @@
     </inertial>
     <visual>
-      <origin xyz="-0.18 0 0.5"/>
+      <origin xyz="-0.18 0 0.05"/>
       <geometry>
         <box size="${BOX_SIZE} ${BOX_SIZE} ${BOX_SIZE}" />
@@ -15,5 +15,5 @@
     </visual>
     <collision>
-      <origin xyz="-0.18 0 0.5"/>
+      <origin xyz="-0.18 0 0.05"/>
       <geometry>
         <box size="${BOX_SIZE} ${BOX_SIZE} ${BOX_SIZE}" />

Commit message: revise ddpg, arm_env etc.

File: as_arm_description/urdf/as_arm.urdf (robot description, URDF)
Before this commit: robot as_arm, 20 links, 19 joints
Links:
- link base_link: mass 1 -> 0.1
- link elbow_link: mass 1 -> 0.1
- link gripper_bottom_link: mass 1 -> 0.1
- link gripper_finger_link1: mass 1 -> 0.1; geometry collision box size=0.01 0.002 0.06; visual box size=0.01 0.002 0.06
- link gripper_finger_link2: mass 1 -> 0.1; geometry collision box size=0.01 0.002 0.06; visual box size=0.01 0.002 0.06
- link gripper_link: mass 1 -> 0.1
- link shoulder_link: mass 1 -> 0.1
- link wrist_flex_link: mass 1 -> 0.1
- link wrist_rot_link: mass 1 -> 0.1
Joints:
- joint finger_joint1: limit lower=-0.015 upper=0 effort=100 velocity=1.0 -> lower=-0.015 upper=0 effort=200 velocity=1.0
- joint finger_joint2: limit lower=0 upper=0.015 effort=100 velocity=1.0 -> lower=0 upper=0.015 effort=200 velocity=1.0

File: as_arm_description/urdf/as_arm.xacro (robot description, xacro)
@@ -16,4 +16,5 @@
     <!-- Constants -->
     <property name="deg_to_rad" value="0.01745329251994329577"/>  <!-- equal to PI/180-->
+    <property name="MATTER_MASS" value="0.1"/>
     <property name="M_SCALE" value="0.001 0.001 0.001"/>
     <property name="M_PI" value="3.14159"/>
@@ -85,5 +86,5 @@
             </geometry>
         </collision>
-        <xacro:inertial_matrix mass="1"/>
+        <xacro:inertial_matrix mass="${MATTER_MASS}"/>
     </link>
     <gazebo reference="base_link">
@@ -113,5 +114,5 @@
             </geometry>
         </collision>
-        <xacro:inertial_matrix mass="1"/>
+        <xacro:inertial_matrix mass="${MATTER_MASS}"/>
     </link>
     <gazebo reference="shoulder_link">
@@ -141,5 +142,5 @@
             </geometry>
         </collision>
-        <xacro:inertial_matrix mass="1"/>
+        <xacro:inertial_matrix mass="${MATTER_MASS}"/>
     </link>
     <gazebo reference="elbow_link">
@@ -169,5 +170,5 @@
             </geometry>
         </collision>
-        <xacro:inertial_matrix mass="1"/>
+        <xacro:inertial_matrix mass="${MATTER_MASS}"/>
     </link>
     <gazebo reference="wrist_flex_link">
@@ -197,5 +198,5 @@
             </geometry>
         </collision>
-        <xacro:inertial_matrix mass="1"/>
+        <xacro:inertial_matrix mass="${MATTER_MASS}"/>
     </link>
     <gazebo reference="wrist_rot_link">
@@ -227,5 +228,5 @@
             </geometry>
         </collision>
-        <xacro:inertial_matrix mass="1"/>
+        <xacro:inertial_matrix mass="${MATTER_MASS}"/>
     </link>
     <gazebo reference="gripper_bottom_link">
@@ -252,5 +253,5 @@
             </geometry>
         </collision>
-        <xacro:inertial_matrix mass="1"/>
+        <xacro:inertial_matrix mass="${MATTER_MASS}"/>
     </link>
     <gazebo reference="gripper_link">
@@ -274,5 +275,11 @@
             <material name="Black"/>
         </visual>
-        <xacro:inertial_matrix mass="0.2"/>
+        <collision>
+            <origin xyz="0 0.016 0.03"/>
+            <geometry>
+                <box size="0.01 0.002 0.06"/>
+            </geometry>
+        </collision>
+        <xacro:inertial_matrix mass="${MATTER_MASS}"/>
     </link>
     <gazebo reference="l_gripper_aft_link">
@@ -296,5 +303,11 @@
             <material name="Black"/>
         </visual>
-        <xacro:inertial_matrix mass="0.2"/>
+        <collision>
+            <origin xyz="0 -0.016 0.03"/>
+            <geometry>
+                <box size="0.01 0.002 0.06"/>
+            </geometry>
+        </collision>
+        <xacro:inertial_matrix mass="${MATTER_MASS}"/>
     </link>
     <gazebo reference="r_gripper_aft_link">
@@ -307,5 +320,5 @@
             <mass value="0.0001"/>
             <cuboid_inertia mass="0.0001" x="0.001" y="0.001" z="0.001"/>
-            <inertia ixx="1.0" ixy="0.0" ixz="0.0" iyy="100.0" iyz="0.0" izz="1.0"/>
+            <inertia ixx="1.0" ixy="0.0" ixz="0.0" iyy="10.0" iyz="0.0" izz="1.0"/>
         </inertial>
         <!--visual>

File: as_arm_description/urdf/object.xacro (robot description, xacro)
@@ -5,5 +5,5 @@
     <inertial>
       <origin xyz="-0.18 0 0" />
-      <mass value="1.0" />
+      <mass value="0.1" />
       <inertia  ixx="1.0" ixy="0.0"  ixz="0.0"  iyy="100.0"  iyz="0.0"  izz="1.0" />
     </inertial>

Commit message: 1. 更改actor 网络的输出层： > 目前actor网络的输出的5个joint的移动角度值，增加一个输出表示cube是否在gripper的抓取范围 > 更改actor网络输出层范围区间为[-4, 4]之间的整数 2. 更改reward计算函数 = exp(-1 * γ * dist(cube, gripper)) 3. 调整摄像头视野，增加摄像头数量，组成双目摄像头 > 提高距离感知，同时避免cube被机械臂遮挡 4. 更改噪音生成函数OuNoice的参数，防止过拟合，探索更多运动空间。 5. 训练阶段： > 第一阶段：一个cube，且cube初始位置不变，gripper初始位置为PreGrasp > 第二阶段：一个cube，且cube初始位置可变，gripper初始位置为PreGrasp > 第三阶段：多个cube，且cube初始位置可变，gripper初始位置为UpRight

File: as_arm_description/urdf/as_arm.urdf (robot description, URDF)
Before this commit: robot as_arm, 20 links, 19 joints
Links:
- added link camera_link_y, mass 1e-5; collision box size=0.01 0.01 0.01; visual box size=0.01 0.01 0.01
- added link camera_mast_link_y; collision box size=0.01 0.01 0.35; visual box size=0.01 0.01 0.35
- added link camera_mast_link_y_2; collision box size=0.15 0.01 0.01; visual box size=0.15 0.01 0.01
- link camera_mast_link: geometry collision box size=0.01 0.01 0.35; visual box size=0.01 0.01 0.35
- link sink_wall_down: geometry collision box size=0.005 0.2 0.025; visual box size=0.005 0.2 0.025
- link sink_wall_left: geometry collision box size=0.2 0.005 0.025; visual box size=0.2 0.005 0.025
- link sink_wall_right: geometry collision box size=0.2 0.005 0.025; visual box size=0.2 0.005 0.025
- link sink_wall_up: geometry collision box size=0.005 0.2 0.025; visual box size=0.005 0.2 0.025
Joints:
- added joint camera_joint_y: type fixed, parent camera_mast_link_y_2, child camera_link_y, origin xyz=-0.14 0 -0.005 rpy=0 1.0471975512 1.57079632679
- added joint camera_mast_joint_y: type fixed, parent bottom_link, child camera_mast_link_y, origin xyz=0 -0.2 0 rpy=0 0 0
- added joint camera_mast_joint_y_2: type fixed, parent camera_mast_link_y, child camera_mast_link_y_2, origin xyz=0 0 0.25 rpy=0 0 0
- joint camera_joint: origin xyz=-0.14 0 -0.005 rpy=0 1.57079632679 0 -> xyz=-0.14 0 -0.005 rpy=0 1.0471975512 -1.57079632679
- joint camera_mast_joint: origin xyz=0 0.1 0 rpy=0 0 0 -> xyz=0 0.2 0 rpy=0 0 0
- joint camera_mast_joint_2: origin xyz=0 0 0.35 rpy=0 0 0 -> xyz=0 0 0.25 rpy=0 0 0

File: as_arm_description/urdf/as_arm.xacro (robot description, xacro)
@@ -21,5 +21,5 @@
     <property name="SINK_WIDTH" value="0.2"/>
     <property name="SINK_WALL_THICK" value="0.005"/>
-    <property name="SINK_DEPTH" value="0.04"/>
+    <property name="SINK_DEPTH" value="0.025"/>
     <!-- Define materials mass -->
     <xacro:macro name="inertial_matrix" params="mass">
@@ -204,4 +204,5 @@
     </gazebo>
     <xacro:include filename="$(find as_arm_description)/urdf/camera.xacro"/>
+    <xacro:include filename="$(find as_arm_description)/urdf/camera_y.xacro"/>
     <xacro:include filename="$(find as_arm_description)/urdf/sink.xacro"/>
     <joint name="wrist_rot_joint" type="revolute">

File: as_arm_description/urdf/camera_y.xacro (robot description, xacro)
@@ -1,11 +1,11 @@
 <?xml version="1.0"?>
 <robot xmlns:xacro="http://www.ros.org/wiki/xacro">
-    <property name="MAST_HEIGHT" value="0.35"/>
-    <joint name="camera_mast_joint" type="fixed">
-        <origin xyz="0 0.2 0" rpy="0 0 0"/>
+    <property name="MAST_HEIGHT_y" value="0.35"/>
+    <joint name="camera_mast_joint_y" type="fixed">
+        <origin xyz="0 -0.2 0" rpy="0 0 0"/>
         <parent link="bottom_link"/>
-        <child link="camera_mast_link"/>
+        <child link="camera_mast_link_y"/>
     </joint>
-    <link name="camera_mast_link">
+    <link name="camera_mast_link_y">
         <visual>
             <origin xyz="0 0 ${MAST_HEIGHT/2-0.02}" rpy="0 0 0"/>
@@ -22,10 +22,10 @@
         </collision>
     </link>
-    <joint name="camera_mast_joint_2" type="fixed">
+    <joint name="camera_mast_joint_y_2" type="fixed">
         <origin xyz="0 0 ${MAST_HEIGHT-0.1}" rpy="0 0 0"/>
-        <parent link="camera_mast_link"/>
-        <child link="camera_mast_link_2"/>
+        <parent link="camera_mast_link_y"/>
+        <child link="camera_mast_link_y_2"/>
     </joint>
-    <link name="camera_mast_link_2">
+    <link name="camera_mast_link_y_2">
         <visual>
             <origin xyz="-0.07 0 0" rpy="0 0 0"/>
@@ -42,11 +42,11 @@
         </collision>
     </link>
-    <joint name="camera_joint" type="fixed">
-        <origin xyz="-0.14 0 -0.005" rpy="0 ${60*deg_to_rad} -${90*deg_to_rad}"/>
-        <parent link="camera_mast_link_2"/>
-        <child link="camera_link"/>
+    <joint name="camera_joint_y" type="fixed">
+        <origin xyz="-0.14 0 -0.005" rpy="0 ${60*deg_to_rad} ${90*deg_to_rad}"/>
+        <parent link="camera_mast_link_y_2"/>
+        <child link="camera_link_y"/>
     </joint>
     <!-- Camera -->
-    <link name="camera_link">
+    <link name="camera_link_y">
         <collision>
             <origin xyz="0 0 -0.005" rpy="0 0 0"/>
@@ -68,20 +68,8 @@
         </inertial>
     </link>
-    <!--joint name="camera_optical_joint" type="fixed">
-        <origin xyz="0 0 0" rpy="0 0 0"/>
-        <parent link="camera_link"/>
-        <child link="camera_optical_link"/>
-    </joint>
-    <link name="camera_optical_link">
-        <inertial>
-            <mass value="1e-5"/>
-            <origin xyz="0 0 0" rpy="${90*deg_to_rad} ${90*deg_to_rad} ${90*deg_to_rad}"/>
-            <inertia ixx="1e-6" ixy="0" ixz="0" iyy="1e-6" iyz="0" izz="1e-6"/>
-        </inertial>
-    </link-->
     <!-- camera -->
-    <gazebo reference="camera_link">
+    <gazebo reference="camera_link_y">
         <material>Gazebo/Red</material>
-        <sensor type="camera" name="camera1">
+        <sensor type="camera" name="camera2">
             <update_rate>30.0</update_rate>
             <camera name="head">
@@ -106,8 +94,8 @@
                 <alwaysOn>true</alwaysOn>
                 <updateRate>0.0</updateRate>
-                <cameraName>camera</cameraName>
+                <cameraName>camera_y</cameraName>
                 <imageTopicName>image_raw</imageTopicName>
                 <cameraInfoTopicName>camera_info</cameraInfoTopicName>
-                <frameName>camera_link</frameName>
+                <frameName>camera_link_y</frameName>
                 <hackBaseline>0.07</hackBaseline>
                 <distortionK1>0.0</distortionK1>

File: as_arm_description/urdf/object.xacro (robot description, xacro)
@@ -1,13 +1,13 @@
 <?xml version="1.0"?>
 <robot name="simple_box" xmlns:xacro="http://www.ros.org/wiki/xacro">
-  <property name="BOX_SIZE" value="0.02"/>
+  <property name="BOX_SIZE" value="0.012"/>
   <link name="cube1">
     <inertial>
       <origin xyz="-0.18 0 0" />
-      <mass value="0.1" />
+      <mass value="0.02" />
       <inertia  ixx="1.0" ixy="0.0"  ixz="0.0"  iyy="100.0"  iyz="0.0"  izz="1.0" />
     </inertial>
     <visual>
-      <origin xyz="-0.18 0 0.05"/>
+      <origin xyz="-0.18 0 0.046"/>
       <geometry>
         <box size="${BOX_SIZE} ${BOX_SIZE} ${BOX_SIZE}" />
@@ -15,5 +15,5 @@
     </visual>
     <collision>
-      <origin xyz="-0.18 0 0.05"/>
+      <origin xyz="-0.18 0 0.046"/>
       <geometry>
         <box size="${BOX_SIZE} ${BOX_SIZE} ${BOX_SIZE}" />
